Commit message: fixed urdf

File: imibot_description/urdf/imibot.urdf (robot description, URDF)
Before this commit: robot imibot, 5 links, 4 joints
Links:
- removed link front_left_wheel
- removed link front_right_wheel
- removed link rear_left_wheel
- removed link rear_right_wheel
- added link front_left_wheel_link; collision cylinder length=0.03 radius=0.032; visual cylinder length=0.03 radius=0.032
- added link front_right_wheel_link; collision cylinder length=0.03 radius=0.032; visual cylinder length=0.03 radius=0.032
- added link rear_left_wheel_link; collision cylinder length=0.03 radius=0.032; visual cylinder length=0.03 radius=0.032
- added link rear_right_wheel_link; collision cylinder length=0.03 radius=0.032; visual cylinder length=0.03 radius=0.032
- link base_link: geometry collision box size=0.255 0.095 0.039; visual box size=0.255 0.095 0.039
Joints:
- removed joint front_left_wheel_joint
- removed joint front_right_wheel_joint
- removed joint rear_left_wheel_joint
- removed joint rear_right_wheel_joint
- added joint front_left_wheel: type continuous, parent base_link, child front_left_wheel_link, origin xyz=-0.065 -0.065 0.032 rpy=0 0 0, axis 0 1 0, limit effort=100 velocity=100
- added joint front_right_wheel: type continuous, parent base_link, child front_right_wheel_link, origin xyz=-0.065 0.065 0.032 rpy=0 0 0, axis 0 1 0, limit effort=100 velocity=100
- added joint rear_left_wheel: type continuous, parent base_link, child rear_left_wheel_link, origin xyz=0.065 -0.065 0.032, axis 0 1 0, limit effort=100 velocity=100
- added joint rear_right_wheel: type continuous, parent base_link, child rear_right_wheel_link, origin xyz=0.065 0.065 0.032 rpy=0 0 0, axis 0 1 0, limit effort=100 velocity=100

File: imibot_description/urdf/imibot.urdf.xacro (robot description, xacro)
@@ -22,5 +22,5 @@
   <!-- Wheel Mounting Positions -->
   <xacro:property name="wheelbase" value="0.11" />
-  <xacro:property name="track" value="0.11" />
+  <xacro:property name="track" value="0.132" />
   <xacro:property name="wheel_vertical_offset" value="0.03282" />
   <!-- Wheel Properties -->
@@ -30,20 +30,17 @@
   <link name="base_link">
     <visual>
-      <origin xyz="0 0 0" rpy="0 0 0" />
+      <origin xyz="0 0 0.032" rpy="0 0 0" />
       <geometry>
         <!--mesh filename="package://imibot_description/meshes/base_link.dae" /-->
-        <box size="0.255 0.1 0.039"/>
+        <box size="${base_x_size} ${base_y_size} ${base_z_size}"/>
       </geometry>
+      <material name="white">
+        <color rgba="1 1 1 1"/>
+      </material>
     </visual>
     <collision>
-      <origin xyz="0 0 ${base_z_size/4}" rpy="0 0 0" />
+      <origin xyz="0 0 0.032" rpy="0 0 0" />
       <geometry>
-        <box size="${base_x_size} ${base_y_size} ${base_z_size/2}"/>
-      </geometry>
-    </collision>
-    <collision>
-      <origin xyz="0 0 ${base_z_size*3/4}" rpy="0 0 0" />
-      <geometry>
-        <box size="${base_x_size*4/5} ${base_y_size} ${base_z_size/2}"/>
+        <box size="${base_x_size} ${base_y_size} ${base_z_size}"/>
       </geometry>
     </collision>
@@ -59,7 +56,7 @@
   <link name="inertial_link">
     <inertial>
-      <mass value="46.034" />
-      <origin xyz="-0.00065 -0.085 0.062" />
-      <inertia ixx="0.6022" ixy="-0.02364" ixz="-0.1197" iyy="1.7386" iyz="-0.001544" izz="2.0296" />
+      <mass value="2" />
+      <origin xyz="0 0 0.032" />
+      <inertia ixx="0.0282916666667" ixy="0" ixz="0" iyy="0.0282916666667" iyz="0" izz="0.05625"/>
     </inertial>
   </link>

File: imibot_description/urdf/wheel.urdf.xacro (robot description, xacro)
@@ -9,9 +9,12 @@
 			</inertial-->
 			<visual>
-				<origin xyz="0 0 0" rpy="0 0 0" />
+				<origin xyz="0 0 0" rpy="${M_PI/2} 0 0" />
 				<geometry>
 					<!--mesh filename="package://imibot_description/meshes/wheel.dae" /-->
-					<cylinder radius="0.032" length="0.03"/>
+					<cylinder radius="${wheel_radius}" length="${wheel_length}"/>
 				</geometry>
+				<material name="black">
+					<color rgba="0 0 0 1"/>
+				</material>
 			</visual>
 			<collision>
