Commit message: changed robot_mg to publish DiffSpeed messages, created DiffSpeed msg, changed imibot_driver to listen on robot_mg and created diff_drive_control_handler.py to use differential speed

File: imibot_description/urdf/imibot.urdf.xacro (robot description, xacro)
@@ -23,8 +23,8 @@
   <xacro:property name="wheelbase" value="0.11" />
   <xacro:property name="track" value="0.132" />
-  <xacro:property name="wheel_vertical_offset" value="0.03282" />
+  <xacro:property name="wheel_vertical_offset" value="0.033" />
   <!-- Wheel Properties -->
   <xacro:property name="wheel_length" value="0.025" />
-  <xacro:property name="wheel_radius" value="0.03282" />
+  <xacro:property name="wheel_radius" value="0.033" />
   <!-- Base link is the center of the robot's bottom plate -->
   <link name="base_link">

Commit message: xtion camera enabled and working

File: imibot_description/urdf/imibot.urdf.xacro (robot description, xacro)
@@ -1,23 +1,22 @@
 <?xml version="1.0"?>
 <robot name="imibot" xmlns:xacro="http://ros.org/wiki/xacro">
-  <!--xacro:arg name="laser_enabled" default="false" />
-  <xacro:arg name="laser_xyz" default="$(optenv imibot_LMS1XX_XYZ 0.2206 0.0 0.00635)" />
-  <xacro:arg name="laser_rpy" default="$(optenv imibot_LMS1XX_RPY 0.0 0.0 0.0)" />
-  <xacro:arg name="kinect_enabled" default="false" />
-  <xacro:arg name="kinect_xyz" default="$(optenv imibot_KINECT_XYZ 0 0 0)" />
-  <xacro:arg name="kinect_rpy" default="$(optenv imibot_KINECT_RPY 0 0.18 3.14)" /-->
+  <xacro:property name="M_PI" value="3.14159"/>
   <xacro:arg name="robot_namespace" default="/" />
-  <!--xacro:arg name="urdf_extras" default="empty.urdf" /-->
-  <!-- Included URDF/XACRO Files -->
-  <!--xacro:include filename="$(find imibot_description)/urdf/decorations.urdf.xacro" /-->
-  <xacro:include filename="$(find imibot_description)/urdf/wheel.urdf.xacro" />
-  <!--xacro:include filename="$(find imibot_description)/urdf/accessories/kinect_camera.urdf.xacro"/>
-  <xacro:include filename="$(find imibot_description)/urdf/accessories/sick_lms1xx_mount.urdf.xacro"/>
-  <xacro:include filename="$(find imibot_description)/urdf/accessories/sensor_arch.urdf.xacro"/-->
-  <xacro:property name="M_PI" value="3.14159"/>
   <!-- Base Size -->
   <xacro:property name="base_x_size" value="0.255" />
   <xacro:property name="base_y_size" value="0.1" />
   <xacro:property name="base_z_size" value="0.039" />
+  <!--xacro:arg name="kinect_enabled" default="false" />
+  <xacro:arg name="kinect_xyz" default="$(optenv imibot_KINECT_XYZ 0 0 0)" />
+  <xacro:arg name="kinect_rpy" default="$(optenv imibot_KINECT_RPY 0 0.18 3.14)" /-->
+  <xacro:arg name="xtion_enabled" default="true" />
+  <xacro:arg name="xtion_xyz" default="$(optenv imibot_XTION_XYZ ${base_x_size/2 - 0.015} 0 ${base_z_size + 0.032})" />
+  <xacro:arg name="xtion_rpy" default="$(optenv imibot_XTION_RPY 0 0 0)" />
+  <!--xacro:arg name="urdf_extras" default="empty.urdf" /-->
+  <!-- Included URDF/XACRO Files -->
+  <xacro:include filename="$(find imibot_description)/urdf/wheel.urdf.xacro" />
+  <xacro:include filename="$(find imibot_description)/urdf/accessories/xtion_camera.urdf.xacro"/>
+  <!--xacro:include filename="$(find imibot_description)/urdf/accessories/kinect_camera.urdf.xacro"/-->
+  <!--xacro:include filename="$(find imibot_description)/urdf/decorations.urdf.xacro" /-->
   <!-- Wheel Mounting Positions -->
   <xacro:property name="wheelbase" value="0.11" />
@@ -30,5 +29,5 @@
   <link name="base_link">
     <visual>
-      <origin xyz="0 0 0.032" rpy="0 0 0" />
+      <origin xyz="0 0 0.032" rpy="0 0 ${M_PI}" />
       <geometry>
         <!--mesh filename="package://imibot_description/meshes/base_link.dae" /-->
@@ -40,5 +39,5 @@
     </visual>
     <collision>
-      <origin xyz="0 0 0.032" rpy="0 0 0" />
+      <origin xyz="0 0 0.032" rpy="0 0 ${M_PI}" />
       <geometry>
         <box size="${base_x_size} ${base_y_size} ${base_z_size}"/>
@@ -47,7 +46,9 @@
   </link>
   <!-- Base footprint is on the ground under the robot -->
-  <link name="base_footprint"/>
+  <link name="base_footprint">
+    <origin rpy="0 0 ${M_PI}" />
+  </link>
   <joint name="base_footprint_joint" type="fixed">
-    <origin xyz="0 0 ${wheel_vertical_offset - wheel_radius}" rpy="0 0 0" />
+    <origin xyz="0 0 ${wheel_vertical_offset - wheel_radius}" rpy="0 0 ${M_PI}" />
     <parent link="base_link" />
     <child link="base_footprint" />
@@ -90,14 +91,5 @@
   </xacro:imibot_wheel>
   <!--xacro:imibot_decorate /-->
-  <!--xacro:if value="$(arg laser_enabled)">
-    <sick_lms1xx_mount prefix="base"/>
-    <sick_lms1xx frame="base_laser" topic="scan" robot_namespace="$(arg robot_namespace)"/>
-    <joint name="laser_mount_joint" type="fixed">
-      <origin xyz="$(arg laser_xyz)" rpy="$(arg laser_rpy)" />
-      <parent link="top_plate_link" />
-      <child link="base_laser_mount" />
-    </joint>
-  </xacro:if>
-  <xacro:if value="$(arg kinect_enabled)">
+  <!--xacro:if value="$(arg kinect_enabled)">
     <xacro:sensor_arch prefix="" parent="top_plate_link">
       <origin xyz="-0.35 0 0.51" rpy="0 0 -3.14"/>
@@ -110,4 +102,12 @@
     <xacro:kinect_camera prefix="camera" robot_namespace="$(arg robot_namespace)"/>
   </xacro:if-->
+  <xacro:if value="$(arg xtion_enabled)">
+    <joint name="xtion_frame_joint" type="fixed">
+      <origin xyz="$(arg xtion_xyz)" rpy="$(arg xtion_rpy)" />
+      <parent link="base_link"/>
+      <child link="camera_link"/>
+    </joint>
+    <xacro:imibot_xtion prefix="camera" robot_namespace="$(arg robot_namespace)"/>
+  </xacro:if>
   <gazebo>
     <plugin name="gazebo_ros_control" filename="libgazebo_ros_control.so">

Commit message: Navigation works fine but odom jumps, trying to incorporate rtabmap

File: imibot_description/urdf/imibot.urdf.xacro (robot description, xacro)
@@ -20,14 +20,14 @@
   <!--xacro:include filename="$(find imibot_description)/urdf/decorations.urdf.xacro" /-->
   <!-- Wheel Mounting Positions -->
-  <xacro:property name="wheelbase" value="0.11" />
-  <xacro:property name="track" value="0.132" />
-  <xacro:property name="wheel_vertical_offset" value="0.033" />
+  <xacro:property name="wheelbase" value="0.111" />
+  <xacro:property name="track" value="0.131" />
+  <xacro:property name="wheel_vertical_offset" value="0.0331" />
   <!-- Wheel Properties -->
-  <xacro:property name="wheel_length" value="0.025" />
-  <xacro:property name="wheel_radius" value="0.033" />
+  <xacro:property name="wheel_length" value="0.0261" />
+  <xacro:property name="wheel_radius" value="0.0331" />
   <!-- Base link is the center of the robot's bottom plate -->
   <link name="base_link">
     <visual>
-      <origin xyz="0 0 0.032" rpy="0 0 ${M_PI}" />
+      <origin xyz="0 0 0.032" rpy="0 0 0" />
       <geometry>
         <!--mesh filename="package://imibot_description/meshes/base_link.dae" /-->
@@ -39,5 +39,5 @@
     </visual>
     <collision>
-      <origin xyz="0 0 0.032" rpy="0 0 ${M_PI}" />
+      <origin xyz="0 0 0.032" rpy="0 0 0" />
       <geometry>
         <box size="${base_x_size} ${base_y_size} ${base_z_size}"/>
@@ -47,8 +47,8 @@
   <!-- Base footprint is on the ground under the robot -->
   <link name="base_footprint">
-    <origin rpy="0 0 ${M_PI}" />
+    <origin rpy="0 0 0" />
   </link>
   <joint name="base_footprint_joint" type="fixed">
-    <origin xyz="0 0 ${wheel_vertical_offset - wheel_radius}" rpy="0 0 ${M_PI}" />
+    <origin xyz="0 0 ${wheel_vertical_offset - wheel_radius}" rpy="0 0 0" />
     <parent link="base_link" />
     <child link="base_footprint" />
@@ -110,5 +110,5 @@
     <xacro:imibot_xtion prefix="camera" robot_namespace="$(arg robot_namespace)"/>
   </xacro:if>
-  <gazebo>
+  <!--gazebo>
     <plugin name="gazebo_ros_control" filename="libgazebo_ros_control.so">
       <robotNamespace>$(arg robot_namespace)</robotNamespace>
@@ -143,5 +143,5 @@
       <drift>0.0001 0.0001 0.0001</drift>
     </plugin>
-  </gazebo>
+  </gazebo-->
   <!-- Optional custom includes. -->
   <!--xacro:include filename="$(arg urdf_extras)" /-->

Commit message: changed urdf

File: imibot_description/urdf/imibot.urdf.xacro (robot description, xacro)
@@ -57,5 +57,5 @@
   <link name="inertial_link">
     <inertial>
-      <mass value="2" />
+      <mass value="3" />
       <origin xyz="0 0 0.032" />
       <inertia ixx="0.0282916666667" ixy="0" ixz="0" iyy="0.0282916666667" iyz="0" izz="0.05625"/>
@@ -69,11 +69,11 @@
   <!-- IMU Link is the standard mounting position for the UM6 IMU.-->
   <!-- Can be modified with environment variables in /etc/ros/setup.bash -->
-  <!--link name="imu_link"/>
+  <link name="imu_link"/>
   <joint name="imu_joint" type="fixed">
-    <origin xyz="$(optenv imibot_IMU_XYZ 0.19 0 0.149)" rpy="$(optenv imibot_IMU_RPY 0 -1.5708 3.1416)" />
+    <origin xyz="$(optenv imibot_IMU_XYZ 0 0 0)" rpy="$(optenv imibot_IMU_RPY 0 0 0)" />
     <parent link="base_link" />
     <child link="imu_link" />
   </joint>
-  <gazebo reference="imu_link">
+  <!--gazebo reference="imu_link">
   </gazebo-->
   <!-- imibot wheel macros -->
